File: mportrai_Bootcamp_Elec/mportrai_Bootcamp_Elec.kicad_sch (KiCad schematic)
At the start: 17 parts, among them J3 FTDI, SW1 SW_Push, U1 ATmega328P-A, Y1 16MHz

Commit message: modif sch-pcb, modif librairie * to mportrai_*, pinout
Parts:
- C1, C2: footprint my_footprints:CL10C120JB8NNNC -> mportrai_footprints:CL10C120JB8NNNC; symbol symbol:Condensateur_12pF -> mportrai_symbol:Condensateur_12pF
- C3, C4, C7: footprint my_footprints:CC0603KRX7R9BB104 -> mportrai_footprints:CC0603KRX7R9BB104; symbol symbol:Condensateur_100nF -> mportrai_symbol:Condensateur_100nF
- C6: footprint my_footprints:CL10A105KB8NNNC -> mportrai_footprints:CL10A105KB8NNNC; symbol symbol:Condensateur_1uF -> mportrai_symbol:Condensateur_1uF
- D1: footprint my_footprints:TZ-P2-0603YGTCS1-0.6T -> mportrai_footprints:TZ-P2-0603YGTCS1-0.6T; symbol symbol:LED_G -> mportrai_symbol:LED_G
- D2: footprint my_footprints:XL-1608SURC-06 -> mportrai_footprints:XL-1608SURC-06; symbol symbol:LED_R -> mportrai_symbol:LED_R
- J1, J2: footprint my_footprints:Connecteur_1 -> mportrai_footprints:Connecteur_1; symbol symbol:Connecteur_1 -> mportrai_symbol:Connecteur_1
- J3: footprint my_footprints:Connecteur_2 -> mportrai_footprints:Connecteur_2; symbol symbol:Connecteur_2 -> mportrai_symbol:Connecteur_2
- R1: footprint my_footprints:0603WAF3300T5E -> mportrai_footprints:0603WAF3300T5E; symbol symbol:Resistance330 -> mportrai_symbol:Resistance330
- R2, R3: footprint my_footprints:RC0603FR-0710KL -> mportrai_footprints:RC0603FR-0710KL; symbol symbol:Resistance10K -> mportrai_symbol:Resistance10K
- SW1: footprint my_footprints:B3U-1000P -> mportrai_footprints:B3U-1000P; symbol symbol:SW_Button -> mportrai_symbol:SW_Button
- U1: footprint my_footprints:ATMEGA328P-AU -> mportrai_footprints:ATMEGA328P-AU; symbol symbol:ATmega328P-A -> mportrai_symbol:ATmega328P-A
- Y1: footprint my_footprints:X322516MLB4SI -> mportrai_footprints:X322516MLB4SI; symbol symbol:Crystal -> mportrai_symbol:Crystal
